File: acmi2-afe.kicad_pcb (KiCad board)
At the start: 6 copper layers, 241.3 x 76.2 mm, 130 parts, among them J1 6469028-1, J2 6469028-1, J3 6469028-1, J4 132134, J5 5499922-4, J6 39301022, J7 5499922-4, Q1 NX7002BKW, T1 T1-1T-KK81, U1 200MHz, U10 TPS3850H50DRCR, U2 LTC2107CUK-PBF, U3 TPS7A8500RGRT, U4 TPSM82866AA0HRDMR, U5 TPS7A8500RGRT, U6 TPS259540DSGR, U7 SN74LVC16T245DGGR, U8 CAT25320VI-GT3

Commit message: added pulser to afe and spi interface for arduino
Parts:
- added C41: 1u, Capacitor_SMD:C_0805_2012Metric, F.Cu at (194.5, 245.5)
- added C42: 10u, Capacitor_SMD:C_0805_2012Metric, F.Cu at (188.2, 248.8)
- added C43: 0.1u, Capacitor_SMD:C_1206_3216Metric, F.Cu at (187.7, 251.5)
- added C47: 0.1u, Capacitor_SMD:C_0805_2012Metric, F.Cu at (215.4, 236.2)
- added C48: 10u, Capacitor_SMD:C_1206_3216Metric, F.Cu at (215.4, 232.7)
- added C49: 0.1u, Capacitor_SMD:C_0805_2012Metric, F.Cu at (230.7, 232.5)
- added C50: 10u, Capacitor_SMD:C_1206_3216Metric, F.Cu at (230.7, 230.3)
- added C51: 0.1u, Capacitor_SMD:C_0805_2012Metric, F.Cu at (215.2, 259.2)
- added C52: 10u, Capacitor_SMD:C_1206_3216Metric, F.Cu at (215.2, 255.2)
- added C53: 0.1u, Capacitor_SMD:C_0805_2012Metric, F.Cu at (230.7, 252.5)
- added C54: 10u, Capacitor_SMD:C_1206_3216Metric, F.Cu at (230.7, 255.0)
- added C55: 0.1u, Capacitor_SMD:C_0805_2012Metric, F.Cu at (215.2, 249.0)
- added C56: 10u, Capacitor_SMD:C_1206_3216Metric, F.Cu at (215.4, 243.7)
- added C57: 0.1u, Capacitor_SMD:C_0805_2012Metric, F.Cu at (230.9, 243.7)
- added C58: 10u, Capacitor_SMD:C_1206_3216Metric, F.Cu at (230.7, 246.5)
- added C59: 1u, Capacitor_SMD:C_0805_2012Metric, F.Cu at (243.0, 230.2)
- added C60: 1u, Capacitor_SMD:C_0805_2012Metric, F.Cu at (243.0, 227.2)
- added C61: 1u, Capacitor_SMD:C_0805_2012Metric, F.Cu at (243.1, 235.7)
- added C62: 1u, Capacitor_SMD:C_0805_2012Metric, F.Cu at (243.0, 233.3)
- added C63: 1u, Capacitor_SMD:C_0805_2012Metric, F.Cu at (243.2, 239.7)
- added C64: 1u, Capacitor_SMD:C_0805_2012Metric, F.Cu at (243.1, 247.7)
- added C65: 1u, Capacitor_SMD:C_0805_2012Metric, F.Cu at (243.1, 245.2)
- added C66: 1u, Capacitor_SMD:C_0805_2012Metric, F.Cu at (243.1, 242.7)
- added C67: 1u, Capacitor_SMD:C_0805_2012Metric, F.Cu at (243.2, 251.7)
- added C68: 1u, Capacitor_SMD:C_0805_2012Metric, F.Cu at (243.2, 254.2)
- added C69: 1u, Capacitor_SMD:C_0805_2012Metric, F.Cu at (264.7, 242.0)
- added C70: 0.1u, Capacitor_SMD:C_0805_2012Metric, F.Cu at (259.7, 233.5)
- added C71: 10u, Capacitor_SMD:C_1206_3216Metric, F.Cu at (259.7, 236.5)
- added C72: 0.1u, Capacitor_SMD:C_0805_2012Metric, F.Cu at (249.2, 246.0)
- added C73: 10u, Capacitor_SMD:C_1206_3216Metric, F.Cu at (249.2, 243.0)
- added CR1: LD1117AS33TR, ld1117as33tr:SOT-223_STM, F.Cu at (189.2, 243.3)
- added J8: 430451202, 430451202:CONN_SD-43045-001_12_MOL, F.Cu at (293.6, 243.7)
- added R28: 49.9, Resistor_SMD:R_0805_2012Metric, F.Cu at (215.3, 246.0)
- added R29: 49.9, Resistor_SMD:R_0805_2012Metric, F.Cu at (234.7, 245.0)
- added R30: 49.9, Resistor_SMD:R_0805_2012Metric, F.Cu at (234.9, 241.7)
- added R31: 49.9, Resistor_SMD:R_0805_2012Metric, F.Cu at (209.3, 252.5)
- added R32: 49.9, Resistor_SMD:R_0805_2012Metric, F.Cu at (209.3, 254.8)
- added R33: 4.02K, Resistor_SMD:R_0805_2012Metric, F.Cu at (239.3, 227.3)
- added R34: 8.06K, Resistor_SMD:R_0805_2012Metric, F.Cu at (239.3, 230.2)
- added R35: 4.02K, Resistor_SMD:R_0805_2012Metric, F.Cu at (239.4, 235.7)
- added R46: 1K, Resistor_SMD:R_0805_2012Metric, F.Cu at (239.3, 233.2)
- added R47: 499, Resistor_SMD:R_0805_2012Metric, F.Cu at (239.4, 239.5)
- added R48: 4.02K, Resistor_SMD:R_0805_2012Metric, F.Cu at (239.4, 247.7)
- added R49: 4.02K, Resistor_SMD:R_0805_2012Metric, F.Cu at (239.4, 245.2)
- added R50: 8.06K, Resistor_SMD:R_0805_2012Metric, F.Cu at (239.4, 242.7)
- added R51: 1K, Resistor_SMD:R_0805_2012Metric, F.Cu at (239.4, 251.7)
- added R52: 499, Resistor_SMD:R_0805_2012Metric, F.Cu at (239.4, 254.2)
- added R53: 19.6K, Resistor_SMD:R_0805_2012Metric, F.Cu at (244.2, 257.3)
- added R54: 300, Resistor_SMD:R_0805_2012Metric, F.Cu at (250.2, 231.7)
- added R55: 2.87K, Resistor_SMD:R_0805_2012Metric, F.Cu at (253.2, 232.6)
- added R56: 0, Resistor_SMD:R_0805_2012Metric, F.Cu at (268.5, 242.0)
- added R57: 0, Resistor_SMD:R_0805_2012Metric, F.Cu at (268.5, 230.5)
- added U11: HFA1412IB, hfa1412ib:SOIC14_4X8P75_INR, F.Cu at (223.7, 232.7)
- added U12: HFA1412IB, hfa1412ib:SOIC14_4X8P75_INR, F.Cu at (223.7, 243.7)
- added U13: HFA1412IB, hfa1412ib:SOIC14_4X8P75_INR, F.Cu at (223.7, 255.0)
- added U14: THS3091D, ths3091d:D8, F.Cu at (252.7, 237.5)
- added U9: SN74LVC827APWR, sn74lvc827:PW24, F.Cu at (197.1, 254.2)
- added XMER1: ADT1-6T+, adt1-6+:CD637_MNC, F.Cu at (268.4, 236.0)
- J5: value 5499922-4 -> 132134; footprint My Footprints:TE_5499922-4 -> Connector_Coaxial:SMA_Amphenol_132134_Vertical
- J6: value 39301022 -> B5B-XH-A; footprint My Footprints:MOLEX_39301022 -> My Footprints:CONN_B5B-XH-A_JST
- moved J6 241.2 mm to (69.4, 231.2)
- moved J5 85.7 mm to (276.2, 221.0)
- moved J4 67.8 mm to (113.7, 221.0)
- moved J7 50.9 mm to (70.2, 297.7), turned to 90 degrees
- moved TP1 46.3 mm to (299.7, 227.5)
- moved MT4 45.9 mm to (246.6, 218.0)
- moved MT6 45.9 mm to (164.7, 218.0)
- moved MT7 45.9 mm to (299.9, 218.0)
- moved MT8 45.9 mm to (68.8, 218.0)
- moved TP4 15.5 mm to (68.2, 254.5)
Connections:
- J3 pad A4: unconnected-(J3-PadA4) -> /Arduino GIGA/giga_sck
- J3 pad B4: unconnected-(J3-PadB4) -> /Arduino GIGA/giga_sdi
- J3 pad C4: unconnected-(J3-PadC4) -> /Arduino GIGA/giga_sdo
- J3 pad D3: unconnected-(J3-PadD3) -> /Arduino GIGA/giga_cs
- J5 pad 1: /Pulser Interface/tp_pos0 -> Net-(J5-In)
- J6 pad 1: GND -> /Arduino GIGA/giga_cs
- J6 pad 2: /Regulators/+5VIN -> /Arduino GIGA/giga_sck
- U6 pad 3: /Regulators/+5VIN -> +5.0V
- U6 pad 4: /Regulators/+5VIN -> +5.0V
Routing:
- net /Arduino GIGA/giga_sck: track 0.00 -> 214.7 mm
- net /Arduino GIGA/giga_cs: track 0.00 -> 211.8 mm
- net /Arduino GIGA/giga_sdi: track 0.00 -> 211.5 mm
- net /Arduino GIGA/giga_sdo: track 0.00 -> 208.2 mm
- net +5.0V: track 36.9 -> 132.1 mm, vias 3 -> 11
- net /Relay Board Interface/spare4: track 126.9 -> 190.5 mm
- net Net-(J4-In): track 8.19 -> 70.5 mm, vias 0 -> 1
- net /Relay Board Interface/spare3: track 133.5 -> 195.2 mm
- net /Relay Board Interface/spare2: track 135.0 -> 194.8 mm
- net /Relay Board Interface/spare1: track 133.5 -> 191.4 mm
- net /Relay Board Interface/spare0: track 133.9 -> 189.9 mm
- net /Relay Board Interface/keylock: track 141.5 -> 195.6 mm
- net /Relay Board Interface/force_trip: track 140.9 -> 193.1 mm
- net -15.0V: track 0.00 -> 50.3 mm, vias 0 -> 1
- net /Relay Board Interface/fault_reset: track 139.2 -> 189.5 mm
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- added copper zone on F.Cu, net +15.0V
- added copper zone on In2.Cu, net +5.0V
- added copper zone on F.Cu, net -15.0V
- added copper zone on In2.Cu, net -5.0V
- removed copper zone on F.Cu, net /Regulators/+5VIN
- removed copper zone on In2.Cu, net GND
Other:
- board size 241.3 x 76.2 mm -> 241.3 x 122.2 mm
- board text added: "NSLS-II ACMI2-AFE SK-2601 Rev 2 10-19-26"
