File: acmi2-afe.kicad_pcb (KiCad board)
At the start: 6 copper layers, 241.3 x 122.2 mm, 188 parts, among them J1 6469028-1, J2 6469028-1, J3 6469028-1, J4 132134, J5 132134, J6 B5B-XH-A, J7 5499922-4, J8 430451202, Q1 NX7002BKW, T1 T1-1T-KK81, U1 200MHz, U10 TPS3850H50DRCR, U11 HFA1412IB, U12 HFA1412IB, U13 HFA1412IB, U14 THS3091D, U2 LTC2107CUK-PBF, U3 TPS7A8500RGRT, U4 TPSM82866AA0HRDMR, U5 TPS7A8500RGRT, U6 TPS259540DSGR, U7 SN74LVC16T245DGGR, U8 CAT25320VI-GT3, U9 SN74LVC827APWR

Commit message: added label for sma connectors
Other:
- board text added: "ICT In"
- board text added: "Test Pulse Out"
