File: acmi2-afe.kicad_sch (KiCad schematic)
At the start: 12 parts

Commit message: added pulser to afe and spi interface for arduino
Other:
- added sheet Arduino GIGA (arduinodisplay.kicad_sch)
- sheet zuDFE Connectors ports: added {arduino_giga}; removed none
Changed lines of the file:
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@@
 		)
 	)
+	(bus
+		(pts
+			(xy 214.63 180.34) (xy 237.49 180.34)
+		)
+		(stroke
+			(width 0)
+			(type default)
+		)
+	)
 	(wire
 		(pts
@@
 	(bus
 		(pts
-			(xy 214.63 161.29) (xy 237.49 161.29)
+			(xy 214.63 151.13) (xy 237.49 151.13)
 		)
 		(stroke
@@
 	(wire
 		(pts
-			(xy 214.63 165.1) (xy 237.49 165.1)
+			(xy 214.63 154.94) (xy 237.49 154.94)
 		)
 		(stroke
@@
 	)
 	(sheet
+		(at 237.49 175.26)
+		(size 27.305 20.955)
+		(exclude_from_sim no)
+		(in_bom yes)
+		(on_board yes)
+		(dnp no)
+		(fields_autoplaced yes)
+		(stroke
+			(width 0.1524)
+			(type solid)
+		)
+		(fill
+			(color 255 255 194 1)
+		)
+		(property "Sheetname" "Arduino GIGA"
+			(at 237.49 174.5484 0)
+			(show_name no)
+			(do_not_autoplace no)
+			(effects
+				(font
+					(size 1.27 1.27)
+				)
+				(justify left bottom)
+			)
+		)
+		(property "Sheetfile" "arduinodisplay.kicad_sch"
+			(at 237.49 196.7996 0)
+			(show_name no)
+			(do_not_autoplace no)
+			(effects
+				(font
+					(size 1.27 1.27)
+				)
+				(justify left top)
+			)
+		)
+		(pin "{arduino_giga}" bidirectional
+			(at 237.49 180.34 180)
+			(effects
+				(font
+					(size 1.27 1.27)
+				)
+				(justify left)
+			)
+		)
+		(instances
+			(project "acmi2-afe"
+				(path "/40891cc8-bf64-41f4-8f69-a607d7b280eb"
+					(page "9")
+				)
+			)
+		)
+	)
+	(sheet
 		(at 124.46 118.11)
 		(size 26.67 24.13)
@@
 		)
 		(pin "{relaybrd}" output
-			(at 214.63 161.29 0)
+			(at 214.63 151.13 0)
 			(effects
 				(font
@@
 		)
 		(pin "wdi" output
-			(at 214.63 165.1 0)
+			(at 214.63 154.94 0)
+			(effects
+				(font
+					(size 1.27 1.27)
+				)
+				(justify right)
+			)
+		)
+		(pin "{arduino_giga}" bidirectional
+			(at 214.63 180.34 0)
 			(effects
 				(font
@@
 	)
 	(sheet
-		(at 237.49 155.575)
+		(at 237.49 145.415)
 		(size 27.305 20.955)
 		(exclude_from_sim no)
@@
 		)
 		(property "Sheetname" "Relay Board Interface"
-			(at 237.49 154.8634 0)
+			(at 237.49 144.7034 0)
 			(show_name no)
 			(do_not_autoplace no)
@@
 		)
 		(property "Sheetfile" "relaybrd.kicad_sch"
-			(at 237.49 177.1146 0)
+			(at 237.49 166.9546 0)
 			(show_name no)
 			(do_not_autoplace no)
@@
 		)
 		(pin "{relaybrd}" output
-			(at 237.49 161.29 180)
+			(at 237.49 151.13 180)
 			(effects
 				(font
@@
 		)
 		(pin "wdi" input
-			(at 237.49 165.1 180)
+			(at 237.49 154.94 180)
 			(effects
 				(font
