File: regulator.kicad_sch (KiCad schematic)
At the start: 37 parts, among them J6 39301022, Q1 NX7002BKW, U3 TPS7A8500RGRT, U4 TPSM82866AA0HRDMR, U5 TPS7A8500RGRT, U6 TPS259540DSGR

Commit message: adding pulser to afe board
Parts:
- removed J6: 39301022, My Footprints:MOLEX_39301022, symbol My Symbols:39301022
- added J8: 430451202, CONN_SD-43045-001_12_MOL, symbol 2026-10-05_18-44-21:430451202
Connections:
- net +5VIN is gone; now on net +5.0V: U6.3 (IN), U6.4 (IN)
- net +5.0V: now also J8.1, J8.7
- net GND: now also J8.10, J8.3, J8.4, J8.9
- new net +15.0V: J8.2, J8.8
- new net -15.0V: J8.12, J8.6
- new net -5.0V: J8.11, J8.5

Commit message: added pulser to afe and spi interface for arduino
Parts:
- J8: footprint CONN_SD-43045-001_12_MOL -> 430451202:CONN_SD-43045-001_12_MOL
Connections:
- net +15.0V: now also J8.1, J8.7; no longer J8.2, J8.8
- net +5.0V: now also J8.2, J8.8; no longer J8.1, J8.7
Changed lines of the file:
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@@
 			)
 		)
-		(property "Footprint" "CONN_SD-43045-001_12_MOL"
+		(property "Footprint" "430451202:CONN_SD-43045-001_12_MOL"
 			(at 303.022 49.53 0)
 			(hide yes)
@@
 			)
 		)
-		(property "Value" "+15.0V"
+		(property "Value" "+5.0V"
 			(at 363.22 62.2299 90)
 			(show_name no)
@@
 			)
 		)
-		(property "Value" "+5.0V"
+		(property "Value" "+15.0V"
 			(at 363.22 59.6899 90)
 			(show_name no)
