File: zudfe_conn.kicad_sch (KiCad schematic)
At the start: 3 parts, among them J1 6469028-1, J2 6469028-1, J3 6469028-1

Commit message: added pulser to afe and spi interface for arduino
Connections:
- net giga_sck: now reaches J3.A4
- net giga_sdi: now reaches J3.B4
- net giga_sdo: now reaches J3.C4
- net giga_cs: now reaches J3.D3
Changed lines of the file:
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@@
 	)
 	(bus_entry
+		(at 320.04 105.41)
+		(size 2.54 2.54)
+		(stroke
+			(width 0)
+			(type default)
+		)
+	)
+	(bus_entry
 		(at 173.99 128.27)
 		(size 2.54 2.54)
@@
 	)
 	(bus_entry
+		(at 320.04 100.33)
+		(size 2.54 2.54)
+		(stroke
+			(width 0)
+			(type default)
+		)
+	)
+	(bus_entry
 		(at 173.99 110.49)
 		(size 2.54 2.54)
@@
 	)
 	(bus_entry
+		(at 320.04 107.95)
+		(size 2.54 2.54)
+		(stroke
+			(width 0)
+			(type default)
+		)
+	)
+	(bus_entry
 		(at 320.04 120.65)
 		(size 2.54 2.54)
@@
 	)
 	(bus_entry
+		(at 320.04 102.87)
+		(size 2.54 2.54)
+		(stroke
+			(width 0)
+			(type default)
+		)
+	)
+	(bus_entry
 		(at 71.12 130.81)
 		(size -2.54 -2.54)
@@
 	(bus
 		(pts
+			(xy 320.04 102.87) (xy 320.04 100.33)
+		)
+		(stroke
+			(width 0)
+			(type default)
+		)
+	)
+	(bus
+		(pts
 			(xy 68.58 125.73) (xy 68.58 123.19)
 		)
@@
 	(bus
 		(pts
-			(xy 320.04 113.03) (xy 320.04 106.68)
+			(xy 320.04 113.03) (xy 320.04 111.76)
 		)
 		(stroke
@@
 		)
 	)
+	(bus
+		(pts
+			(xy 320.04 105.41) (xy 320.04 102.87)
+		)
+		(stroke
+			(width 0)
+			(type default)
+		)
+	)
 	(wire
 		(pts
@@
 	(wire
 		(pts
+			(xy 322.58 107.95) (xy 337.82 107.95)
+		)
+		(stroke
+			(width 0)
+			(type default)
+		)
+	)
+	(wire
+		(pts
 			(xy 337.82 148.59) (xy 322.58 148.59)
 		)
@@
 	(wire
 		(pts
+			(xy 322.58 105.41) (xy 337.82 105.41)
+		)
+		(stroke
+			(width 0)
+			(type default)
+		)
+	)
+	(wire
+		(pts
 			(xy 322.58 125.73) (xy 337.82 125.73)
 		)
@@
 		)
 	)
+	(wire
+		(pts
+			(xy 322.58 110.49) (xy 337.82 110.49)
+		)
+		(stroke
+			(width 0)
+			(type default)
+		)
+	)
 	(bus
 		(pts
@@
 	(bus
 		(pts
-			(xy 308.61 106.68) (xy 320.04 106.68)
+			(xy 308.61 111.76) (xy 320.04 111.76)
+		)
+		(stroke
+			(width 0)
+			(type default)
+		)
+	)
+	(wire
+		(pts
+			(xy 322.58 102.87) (xy 337.82 102.87)
 		)
 		(stroke
@@
 		)
 	)
+	(bus
+		(pts
+			(xy 320.04 100.33) (xy 320.04 97.79)
+		)
+		(stroke
+			(width 0)
+			(type default)
+		)
+	)
 	(wire
 		(pts
@@
 		)
 	)
+	(bus
+		(pts
+			(xy 320.04 107.95) (xy 320.04 105.41)
+		)
+		(stroke
+			(width 0)
+			(type default)
+		)
+	)
 	(wire
 		(pts
@@
 		)
 	)
+	(bus
+		(pts
+			(xy 308.61 97.79) (xy 320.04 97.79)
+		)
+		(stroke
+			(width 0)
+			(type default)
+		)
+	)
 	(wire
 		(pts
@@
 		)
 	)
+	(label "giga_sck"
+		(at 327.66 105.41 0)
+		(effects
+			(font
+				(size 1.27 1.27)
+			)
+			(justify left bottom)
+		)
+	)
 	(label "fault_led6"
 		(at 179.07 143.51 0)
@@
 		)
 	)
+	(label "giga_sdo"
+		(at 327.66 110.49 0)
+		(effects
+			(font
+				(size 1.27 1.27)
+			)
+			(justify left bottom)
+		)
+	)
 	(label "fault_led1"
 		(at 180.34 171.45 0)
@@
 		)
 	)
+	(label "giga_sdi"
+		(at 327.66 107.95 0)
+		(effects
+			(font
+				(size 1.27 1.27)
+			)
+			(justify left bottom)
+		)
+	)
 	(label "D8_N"
 		(at 82.55 123.19 180)
@@
 		)
 	)
+	(label "giga_cs"
+		(at 327.66 102.87 0)
+		(effects
+			(font
+				(size 1.27 1.27)
+			)
+			(justify left bottom)
+		)
+	)
 	(label "tp_pos1"
 		(at 334.01 95.25 180)
@@
 		)
 	)
+	(hierarchical_label "{arduino_giga}"
+		(shape bidirectional)
+		(at 308.61 97.79 180)
+		(effects
+			(font
+				(size 1.27 1.27)
+			)
+			(justify right)
+		)
+	)
 	(hierarchical_label "{ADC}"
 		(shape bidirectional)
@@
 	(hierarchical_label "{eeprom}"
 		(shape input)
-		(at 308.61 106.68 180)
+		(at 308.61 111.76 180)
 		(effects
 			(font
